File: PCB-Keychains.kicad_pcb (KiCad board)
At the start: 2 copper layers, 278.1 x 182.9 mm, 1519 parts

Commit message: Add readme
Parts:
- added G***: LOGO, locallib:ai-ring-6mm-Combined, B.Cu at (187.6, 97.6)
- added G***: LOGO, locallib:ai-ring-6mm-Combined, B.Cu at (170.0, 125.7)
- added G***: LOGO, locallib:ai-ring-6mm-Combined, B.Cu at (211.9, 159.5)
- added G***: LOGO, locallib:ai-ring-6mm-Combined, B.Cu at (211.9, 183.4)
- added G***: LOGO, locallib:ai-ring-6mm-Combined, B.Cu at (209.1, 127.2)
- added G***: LOGO, locallib:ai-ring-6mm-Combined, B.Cu at (279.6, 127.2)
- added G***: LOGO, locallib:ai-ring-6mm-Combined, B.Cu at (219.6, 55.7)
- added G***: LOGO, locallib:ai-ring-6mm-Combined, B.Cu at (269.1, 55.7)
- added G***: LOGO, locallib:ai-ring-6mm-Combined, B.Cu at (165.3, 55.7)
- added G***: LOGO, locallib:ai-ring-6mm-Combined, B.Cu at (95.7, 64.3)
- added G***: LOGO, locallib:ai-ring-6mm-Combined, B.Cu at (17.6, 64.3)
- added G***: LOGO, locallib:ai-ring-6mm-Combined, B.Cu at (100.5, 98.1)
- added G***: LOGO, locallib:ai-ring-6mm-Combined, B.Cu at (17.6, 31.9)
- added G***: LOGO, locallib:ai-ring-6mm-Combined, B.Cu at (84.3, 31.9)
- added G***: LOGO, locallib:ai-ring-6mm-Combined, B.Cu at (155.7, 31.9)
- added G***: LOGO, locallib:ai-ring-6mm-Combined, B.Cu at (225.3, 31.9)
- added G***: LOGO, locallib:ai-ring-6mm-Combined, B.Cu at (17.6, 99.5)
- added G***: LOGO, locallib:ai-ring-6mm-Combined, B.Cu at (17.6, 127.2)
- added G***: LOGO, locallib:ai-ring-6mm-Combined, B.Cu at (17.6, 159.5)
- added G***: LOGO, locallib:ai-ring-6mm-Combined, B.Cu at (17.6, 191.0)
- added G***: LOGO, locallib:ai-ring-6mm-Combined, B.Cu at (111.9, 178.6)
- added G***: LOGO, locallib:ai-ring-6mm-Combined, B.Cu at (111.9, 151.0)
- added G***: LOGO, locallib:ai-ring-6mm-Combined, B.Cu at (104.3, 125.7)
Other:
- outline, holes or cut-outs redrawn
- board text added: "Mechanical Keyboards Numpad"
